File: electronics/pilkki.kicad_sch (KiCad schematic)
At the start: 59 parts, among them J1 USB_C_Receptacle, J2 Conn_01x01_Pin, J3 Conn_01x08, J4 Conn_01x10, Q1 SSM6N35AFE, Q2 DMG1023UV, SW1 EVQ-P2202M, U2 MIC23050-SYML, U2 TPD2EUSB30A, U3 STM32G431KBUx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

Commit message: Update pilkki.kicad_sch
Other:
- company: Alzymologist Oy -> Kalapaja Oy
Changed lines of the file:
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@@
     (date "2023-07-18")
     (rev ".1A")
-    (company "Alzymologist Oy")
+    (company "Kalapaja Oy")
   )
   (junction (at 83.82 22.86) (diameter 0) (color 0 0 0 0)
